File: AOML_AB_3.0/untitled.kicad_sch (KiCad schematic)
At the start: 28 parts, among them IC1 CD4043BDR, IC2 CD4043BDR, J5 Conn_01x03, K1 TX2-L2-5V, K10 TX2-L2-5V, K11 TX2-L2-5V, K12 TX2-L2-5V, K13 TX2-L2-5V, K2 TX2-L2-5V, K3 TX2-L2-5V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

Commit message: relays & ssr finished / MAX3232 finished
Parts:
- added R3, R4, R5, R6, R7, R8, R9: 320, symbol Device:R
- added U10, U11, U12, U13, U14, U9: TLP170AM, Package_SO:MFSOP6-4_4.4x3.6mm_P1.27mm, symbol Relay_SolidState:TLP175A
- R2: value R -> 320
Connections:
- net GND: now also IC1.8 (VSS), IC2.8 (VSS), R3.2, R4.2, R5.2, R6.2, R7.2, R8.2, R9.2
- net Reset1: now also IC1.11 (R3), IC1.15 (R4), IC1.3 (R1), IC1.7 (R2)
- net Reset2: now also IC2.11 (R3), IC2.15 (R4), IC2.3 (R1), IC2.7 (R2)
- net XBT1_C: now also U8.4
- net XBT2_C: now also U7.4
- net XBT3_C: now also U9.4
- net XBT4_C: now also U10.4
- net XBT5_C: now also U11.4
- net XBT6_C: now also U12.4
- net XBT7_C: now also U13.4
- net XBT8_C: now also U14.4
- net at IC1.1 (Q4): now also U7.1; no longer U8.1
- net at IC1.10 (Q3): now also U9.1
- net SSR_xbt3: now reaches IC1.12 (S3)
- net SSR_xbt2: now reaches IC1.14 (S4)
- net +3.3V: now reaches IC1.16 (VDD)
- net +3.3V: now also IC1.5 (ENABLE), IC2.16 (VDD), IC2.5 (ENABLE)
- net at IC1.2 (Q1): now also U8.1; no longer U7.1
- net SSR_xbt1: now reaches IC1.4 (S1)
- net SSR_xbt4: now reaches IC1.6 (S2)
- net at IC1.9 (Q2): now also U10.1
- net relay_xbt8: now reaches U6.1 (I1)
- net relay_gnd-cond: now reaches U6.2 (I2)
- net relay_cal-cont: now reaches U6.3 (I3)
- net relay_cal-res: now reaches U6.4 (I4)
- net relay_reset1: now reaches U6.5 (I5)
- net relay_reset2: now reaches U6.6 (I6)
- net relay_reset3: now reaches U6.7 (I7)
- net C: now reaches U7.6
- net C: now also U8.6, U10.6, U11.6, U12.6, U13.6, U14.6, U9.6
- net at U8.3: now also R3.1
- net at IC2.1 (Q4): now also U12.1
- net at IC2.10 (Q3): now also U13.1
- net SSR_xbt7: now reaches IC2.12 (S3)
- net SSR_xbt6: now reaches IC2.14 (S4)
- net at IC2.2 (Q1): now also U11.1
- net SSR_xbt5: now reaches IC2.4 (S1)
- net SSR_xbt8: now reaches IC2.6 (S2)
- net at IC2.9 (Q2): now also U14.1
- net relay_xbt1: now reaches U5.1 (I1)
- net relay_xbt2: now reaches U5.2 (I2)
- net relay_xbt3: now reaches U5.3 (I3)
- net relay_xbt4: now reaches U5.4 (I4)
- net relay_xbt5: now reaches U5.5 (I5)
- net relay_xbt6: now reaches U5.6 (I6)
- net relay_xbt7: now reaches U5.7 (I7)
- new net: R6.1, U11.3
- new net: R4.1, U9.3
- new net: R8.1, U13.3
- new net: R5.1, U10.3
- new net: R7.1, U12.3
- new net: R9.1, U14.3
Other:
- note added: "R-ON max = 0.3 ohm"
- note added: "Reset 1-2-3-4"
- note added: "Reset 5-6-7-8"
- note added: "To MK21"
- moved on the sheet: IC1, J5, K1, K10, K11, K12, K13, K2, K3, K4, K5, K6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
