File: AOML_AB_3.0/AOML_AB_3.0.kicad_pcb (KiCad board)
At the start: 2 copper layers, 194 parts, among them IC1 CD4043BDR, IC10 DRV8825PWPR, IC2 CD4043BDR, IC3 DRV8825PWPR, IC4 DRV8825PWPR, IC5 DRV8825PWPR, IC6 DRV8825PWPR, IC7 DRV8825PWPR, IC8 DRV8825PWPR, IC9 DRV8825PWPR, J1 216550-1, J10 Conn_01x03, J11 Conn_01x03, J12 Conn_01x03, J13 Screw_Terminal_01x07, J14 216548-1, J15 216548-1, J16 216548-1, J17 216548-1, J18 216548-1, J19 216548-1, J2 Conn_01x04, J20 216548-1, J21 216548-1, J22 Screw_Terminal_01x05, J23 Screw_Terminal_01x04, J3 Conn_01x03, J4 Screw_Terminal_01x04, J5 Conn_01x03, J6 Conn_01x03, J7 Conn_01x03, J8 Conn_01x03, J9 Conn_01x03, K1 TX2-L2-5V, K10 TX2-L2-5V, K11 TX2-L2-5V, K12 TX2-L2-5V, K2 TX2-L2-5V, K3 TX2-L2-5V, K4 TX2-L2-5V, K5 TX2-L2-5V, K6 TX2-L2-5V, K7 TX2-L2-5V, K8 TX2-L2-5V, K9 TX2-L2-5V, SW1 TS02-66-70-BK-160-LCR-D, SW2 SW_DIP_x03, U1 INA213AIDCKR, U10 TLP170AM, U11 TLP170AM, U12 TLP170AM, U13 TLP170AM, U14 TLP170AM, U15 MAX3232, U16 AT24C01D-STUM-T, U17 L7812ABD2T-TR, U2 STM32F103RBTx, U3 LM7805MPX, U4 MCP1825ST-3302E/DB, U5 ULN2003ADR, U6 ULN2003ADR, U7 TLP170AM, U8 TLP170AM, U9 TLP170AM, Y1 8MHz

Commit message: PBC edge and final footprint review, jlpcb restrictions revised
Parts:
- added REF**: MountingHole_2.5mm_Pad, MountingHole:MountingHole_2.5mm_Pad, F.Cu at (48.0, 43.0)
- added REF**: MountingHole_2.5mm_Pad, MountingHole:MountingHole_2.5mm_Pad, F.Cu at (48.0, 131.0)
- added REF**: MountingHole_2.5mm_Pad, MountingHole:MountingHole_2.5mm_Pad, F.Cu at (197.0, 43.0)
- added REF**: MountingHole_2.5mm_Pad, MountingHole:MountingHole_2.5mm_Pad, F.Cu at (197.0, 131.0)
- C5: renamed from C1; footprint Capacitor_1000uF:CAP_PAN_12.5X25_PAN -> Capacitor_1000uF_can-smt:CAP_EEV_H13_PAN
- RN4: footprint Resistor_THT:R_Array_SIP9 -> Resistor_network-330:RESCAV80P400X210X65-10N
- moved K7 350.5 mm to (431.8, 243.8)
- moved K6 341.2 mm to (411.5, 243.8)
- moved R10 315.2 mm to (421.6, 264.2)
- moved R11 314.0 mm to (412.8, 269.2)
- moved K5 294.9 mm to (342.9, 243.8)
- moved K12 284.5 mm to (370.8, 243.8)
- moved JP8 276.9 mm to (382.3, 248.9)
- moved J8 272.2 mm to (0.92, 277.4)
- moved U10 268.1 mm to (12.1, 255.3)
- moved JP7 256.3 mm to (354.4, 248.9)
- moved J14 255.7 mm to (297.6, 277.4)
- moved U11 252.0 mm to (52.7, 255.3)
- moved K1 251.6 mm to (-5.08, 243.8)
- moved J15 248.5 mm to (42.0, 277.4)
- moved JP6 241.0 mm to (331.4, 248.9)
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- renumbered C3 to C1, C17 to C10, C13 to C11, C2 to C12, C7 to C13, C9 to C14, C26 to C15, C14 to C16, C4 to C17, C6 to C18, C10 to C19, C5 to C2, C33 to C21, C23 to C22, C21 to C23, C25 to C24, C24 to C25, C35 to C26, C18 to C27, C19 to C28, C34 to C29, C8 to C3, C28 to C30, C48 to C31, C66 to C32, C31 to C33, C27 to C34, C49 to C35, C50 to C36, C67 to C37, C68 to C38, C29 to C39, C15 to C4, C51 to C40, C69 to C41, C30 to C42, C52 to C43, C70 to C44, C32 to C45, C53 to C46, C71 to C47, C36 to C48, C54 to C49, C72 to C50, C37 to C51, C38 to C52, C55 to C53, C56 to C54, C73 to C55, C74 to C56, C39 to C57, C57 to C58, C75 to C59, C11 to C6, C40 to C60, C58 to C61, C76 to C62, C41 to C63, C59 to C64, C77 to C65, C42 to C66, C60 to C67, C43 to C68, C44 to C69, C16 to C7, C61 to C70, C62 to C71, C45 to C72, C63 to C73, C46 to C74, C64 to C75, C47 to C76, C65 to C77, C22 to C8, C12 to C9, D2 to D1, D1 to D2, IC8 to IC10, IC6 to IC4, IC9 to IC5, IC4 to IC6, IC10 to IC8, IC5 to IC9, J2 to J1, J9 to J10, J8 to J12, J10 to J13, J12 to J14, J6 to J15, J15 to J16, J20 to J18, J14 to J19, J1 to J2, J18 to J20, J16 to J22, J19 to J23, J4 to J3, J22 to J4, J23 to J5, J3 to J6, J13 to J7, J5 to J8, J7 to J9, JP6 to JP1, JP8 to JP2, JP7 to JP3, JP1 to JP6, JP2 to JP7, JP3 to JP8, R37 to R1, R2 to R10, R3 to R11, R9 to R12, R18 to R13, R27 to R14, R8 to R15, R19 to R16, R28 to R17, R12 to R18, R20 to R19, R36 to R2, R29 to R20, R11 to R21, R21 to R22, R30 to R23, R13 to R24, R22 to R25, R31 to R26, R14 to R27, R23 to R28, R32 to R29, R38 to R3, R15 to R30, R24 to R31, R16 to R32, R25 to R33, R17 to R34, R26 to R35, R39 to R4, R4 to R5, R1 to R6, R6 to R7, R5 to R8, R7 to R9, RN2 to RN1, RN3 to RN2, RN1 to RN3, RV9 to RV1, U17 to U1, U8 to U10, U7 to U11, U9 to U12, U10 to U13, U11 to U14, U12 to U15, U13 to U16, U14 to U17, U3 to U2, U4 to U3, U15 to U4, U1 to U5, U2 to U6, U16 to U7, U5 to U8, U6 to U9
Other:
- board outline added: 310 x 100 mm

Commit message: PCB layout finished, next step is routing
Parts:
- removed REF** (x4): MountingHole_2.5mm_Pad, MountingHole:MountingHole_2.5mm_Pad
- added H1: MountingHole, MountingHole:MountingHole_2.5mm_Pad, F.Cu at (59.0, 92.5)
- added H2: MountingHole, MountingHole:MountingHole_2.5mm_Pad, F.Cu at (208.0, 92.5)
- added H3: MountingHole, MountingHole:MountingHole_2.5mm_Pad, F.Cu at (59.0, 180.5)
- added H4: MountingHole, MountingHole:MountingHole_2.5mm_Pad, F.Cu at (208.0, 180.5)
- added H5: MountingHole, MountingHole:MountingHole_2.5mm_Pad, F.Cu at (357.0, 92.5)
- added H6: MountingHole, MountingHole:MountingHole_2.5mm_Pad, F.Cu at (357.0, 180.5)
- added RN5: R_Pack04, Resistor_network_x4_-330:RESCAXE80P320X160X70-8N, F.Cu at (209.0, 112.3)
- C10: footprint Capacitor_1uF:CAP_WCAP-ATG5_05.0X11.0_WRE -> Capacitor_1uF-ceramic:CAP_CL21_SAM
- RN4: value 330 -> R_Pack04; footprint Resistor_network-330:RESCAV80P400X210X65-10N -> Resistor_network_x4_-330:RESCAXE80P320X160X70-8N
- moved RV1 270.9 mm to (86.0, 177.5), turned to -90 degrees
- moved SW2 269.7 mm to (71.8, 178.8), turned to -90 degrees
- moved J17 258.7 mm to (195.2, 171.0), turned to 180 degrees
- moved J20 257.1 mm to (227.3, 171.0), turned to 180 degrees
- moved J23 255.5 mm to (257.2, 171.0), turned to 180 degrees
- moved J19 254.9 mm to (135.6, 171.0), turned to 180 degrees
- moved J22 254.5 mm to (165.4, 171.0), turned to 180 degrees
- moved J16 252.6 mm to (105.8, 171.0), turned to 180 degrees
- moved J18 250.3 mm to (287.2, 171.0), turned to 180 degrees
- moved J21 249.8 mm to (317.2, 171.0), turned to 180 degrees
- moved J5 244.2 mm to (296.5, 104.5)
- moved R19 239.1 mm to (183.0, 161.5)
- moved C40 238.9 mm to (183.0, 158.9), turned to 180 degrees
- moved IC4 238.7 mm to (192.0, 161.5)
- moved C43 238.5 mm to (183.0, 156.4)
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Connections:
- C10 pad 1: GND -> /VDDA
- C7 pad 1: GND -> /VDDA
- FB1 pad 2: GND -> /VDDA
- RN4 pad 2: Net-(RN4-R1) -> GND
- RN4 pad 3: Net-(RN4-R2) -> GND
- RN4 pad 4: Net-(RN4-R3) -> GND
- RN4 pad 5: Net-(RN4-R4) -> Net-(RN4-R4.2)
- RN4 pad 6: Net-(RN4-R5) -> Net-(RN4-R3.2)
- RN4 pad 7: Net-(RN4-R6) -> Net-(RN4-R2.2)
- RN4 pad 8: Net-(RN4-R7) -> Net-(RN4-R1.2)
- U10 pad 3: Net-(RN4-R8) -> Net-(RN4-R1.2)
- U11 pad 3: Net-(RN4-R7) -> Net-(RN4-R2.2)
- U12 pad 3: Net-(RN4-R6) -> Net-(RN4-R3.2)
- U13 pad 3: Net-(RN4-R5) -> Net-(RN4-R4.2)
- U14 pad 3: Net-(RN4-R4) -> Net-(RN5-R1.2)
- U15 pad 3: Net-(RN4-R3) -> Net-(RN5-R2.2)
- U16 pad 3: Net-(RN4-R2) -> Net-(RN5-R3.2)
- U17 pad 3: Net-(RN4-R1) -> Net-(RN5-R4.2)
- U6 pad 13: GND -> /VDDA
Other:
- board text added: "eeprom"

Commit message: PCB reorganized for better routing, R networks changed to x4, power leds added, micro outputs need relocation to allow easier routing to each side
Parts:
- removed RN5: R_Pack04, Resistor_network_x4_-330:RESCAXE80P320X160X70-8N
- added D4: green, LED_green_0603:LED_B1911PG--20D000514U1930_HVK, F.Cu at (90.6, 159.0)
- added D5: green, LED_green_0603:LED_B1911PG--20D000514U1930_HVK, F.Cu at (85.4, 123.0)
- added D6: green, LED_green_0603:LED_B1911PG--20D000514U1930_HVK, F.Cu at (126.0, 141.0)
- added JP10: SolderJumper_2_Open, Jumper:SolderJumper-2_P1.3mm_Open_RoundedPad1.0x1.5mm, F.Cu at (231.3, 130.0)
- added JP9: SolderJumper_2_Open, Jumper:SolderJumper-2_P1.3mm_Open_RoundedPad1.0x1.5mm, F.Cu at (231.3, 140.0)
- added R36: 330, Resistor_0805:RC0805N_YAG, F.Cu at (240.0, 113.0)
- added R37: 330, Resistor_0805:RC0805N_YAG, F.Cu at (217.0, 113.0)
- added R38: 330, Resistor_0805:RC0805N_YAG, F.Cu at (184.0, 113.0)
- added R39: 330, Resistor_0805:RC0805N_YAG, F.Cu at (161.1, 111.0)
- added R40: 330, Resistor_0805:RC0805N_YAG, F.Cu at (138.1, 112.0)
- added R41: 330, Resistor_0805:RC0805N_YAG, F.Cu at (114.7, 113.0)
- added R42: 330, Resistor_0805:RC0805N_YAG, F.Cu at (92.0, 113.1)
- added R43: 330, Resistor_0805:RC0805N_YAG, F.Cu at (69.3, 113.0)
- added R44: 2k, Resistor_0805:RC0805N_YAG, F.Cu at (90.9, 161.0)
- added R45: 560, Resistor_0805:RC0805N_YAG, F.Cu at (85.1, 125.0)
- added R46: 220, Resistor_0805:RC0805N_YAG, F.Cu at (126.2, 143.0)
- RN2: footprint Resistor_network-10k:SMT_JR-0710KL_YAG -> Resistor_network_x4_10k-1204:RESCAXS80P320X160X70-8N
- RN4: value R_Pack04 -> 10k; footprint Resistor_network_x4_-330:RESCAXE80P320X160X70-8N -> Resistor_network_x4_10k-1204:RESCAXS80P320X160X70-8N
- SW1: footprint Button_TS02_66_70_BK_160_LCR_D:SW_TS02-66-70-BK-160-LCR-D -> Button_switch_smt:SMT_FS
- Y1: footprint Oscillator_8mhz_ECS-80-18-4X-CKM:ECS80184XCKM -> Crystal_8MHZ_smt:XTAL_ABLS-8.000MHz-20-B-3-H-T
- moved C29 153.8 mm to (334.1, 125.0)
- moved R9 153.8 mm to (334.1, 122.0)
- moved C22 88.0 mm to (195.6, 136.6)
- moved C8 88.0 mm to (195.6, 134.1)
- moved C15 88.0 mm to (210.0, 132.4)
- moved C24 88.0 mm to (203.0, 141.4)
- moved C25 88.0 mm to (203.0, 130.6)
- moved U4 88.0 mm to (203.0, 136.0)
- moved R2 38.9 mm to (334.1, 112.0)
- moved R1 38.8 mm to (334.1, 115.0)
- moved C28 29.0 mm to (229.1, 135.1)
- moved R7 29.0 mm to (224.0, 130.6)
- moved R8 29.0 mm to (224.0, 139.6)
- moved U7 29.0 mm to (223.9, 135.1)
- moved C3 23.2 mm to (117.2, 146.0)
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Connections:
- C28 pad 1: +3.3V -> Net-(JP9-A)
- IC1 pad 11: /RelayControl/Reset1 -> relay_reset1
- IC1 pad 15: /RelayControl/Reset1 -> relay_reset1
- IC1 pad 3: /RelayControl/Reset1 -> relay_reset1
- IC1 pad 7: /RelayControl/Reset1 -> relay_reset1
- IC2 pad 11: /RelayControl/Reset2 -> relay_reset2
- IC2 pad 15: /RelayControl/Reset2 -> relay_reset2
- IC2 pad 3: /RelayControl/Reset2 -> relay_reset2
- IC2 pad 7: /RelayControl/Reset2 -> relay_reset2
- RN1 pad 3: unconnected-(RN1-R2-Pad3) -> relay_reset3
- RN1 pad 4: relay_reset3 -> relay_reset2
- RN1 pad 5: relay_reset2 -> relay_reset1
- RN1 pad 6: relay_reset1 -> relay_cal_res
- RN1 pad 7: relay_cal_res -> relay_cal_cont
- RN1 pad 8: relay_cal_cont -> relay_gnd_cond
- RN1 pad 9: relay_gnd_cond -> relay_xbt8
- RN2 pad 2: SSR_xbt8 -> GND
- RN2 pad 3: SSR_xbt7 -> GND
- RN2 pad 4: SSR_xbt6 -> GND
- RN2 pad 5: SSR_xbt5 -> SSR_xbt8
- RN2 pad 6: SSR_xbt4 -> SSR_xbt7
- RN2 pad 7: SSR_xbt3 -> SSR_xbt6
- RN2 pad 8: SSR_xbt2 -> SSR_xbt5
- RN3 pad 2: relay_xbt8 -> unconnected-(RN3-R1-Pad2)
- RN4 pad 5: Net-(RN4-R4.2) -> SSR_xbt4
- RN4 pad 6: Net-(RN4-R3.2) -> SSR_xbt3
- RN4 pad 7: Net-(RN4-R2.2) -> SSR_xbt2
- RN4 pad 8: Net-(RN4-R1.2) -> SSR_xbt1
- U10 pad 3: Net-(RN4-R1.2) -> Net-(R43-Pad1)
- U11 pad 3: Net-(RN4-R2.2) -> Net-(R42-Pad1)
- U12 pad 3: Net-(RN4-R3.2) -> Net-(R41-Pad1)
- U13 pad 3: Net-(RN4-R4.2) -> Net-(R40-Pad1)
- U7 pad 4: +3.3V -> Net-(JP9-A)
- U7 pad 5: GND -> Net-(JP10-A)
Other:
- board text added: "12V Vreg"
- board text added: "3V3 Vreg"
- board text added: "5V Vreg"
- board text added: "Aux GPIO"
- board text added: "Auxiliary: GND & Calibration"
- board text added: "LCD & local control"
- board text added: "Microcontroller"
- board text added: "Motor control"
- board text added: "Motor current"
- board text added: "STM32 UART3 3V3 AXR UART 5V"
- board text added: "TTL RS232"
- board text added: "UART2/RS232 gps"
- board text added: "Vin to ADC"
- board text added: "WP"

Commit message: Microcontroller pin connections reorganized, test back ground plane routed
Parts:
- added J24: Conn_01x06, Connector_PinHeader_2.54mm:PinHeader_1x06_P2.54mm_Vertical, F.Cu at (344.0, 148.9)
- added JP11: SolderJumper_2_Open, Jumper:SolderJumper-2_P1.3mm_Open_RoundedPad1.0x1.5mm, F.Cu at (83.4, 167.7)
- J4: value Screw_Terminal_01x05 -> PH2-08-UA; footprint Header_screw_5x1_TB003-500-P05BE:CUI_TB003-500-P05BE -> Connector_PinHeader_2.54mm:PinHeader_2x04_P2.54mm_Vertical
- J6: footprint Header_male_3x1_jumper:CONN03_6130_7P62X2P54_WRE -> Connector_PinHeader_2.54mm:PinHeader_1x03_P2.54mm_Vertical
- moved J4 271.3 mm to (76.5, 130.4), turned to 0 degrees
- moved RV1 240.3 mm to (322.2, 131.5), turned to 90 degrees
- moved SW2 240.3 mm to (308.0, 134.5), turned to 180 degrees
- moved R6 26.7 mm to (153.1, 115.5)
- moved J6 24.5 mm to (146.9, 119.5), turned to 0 degrees
- moved C27 14.8 mm to (120.1, 122.5)
- moved SW1 8.05 mm to (127.8, 122.6)
- moved D1 7.15 mm to (77.1, 143.4)
- moved C4 7.02 mm to (138.0, 121.5)
- moved J1 6.48 mm to (168.5, 119.5)
- moved C26 6.13 mm to (87.0, 171.8)
- moved C6 3.05 mm to (151.1, 124.1)
- moved C5 3.00 mm to (98.0, 136.5)
- moved C21 2.05 mm to (159.1, 115.5)
- moved D3 1.94 mm to (80.0, 172.2)
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Connections:
- C26 pad 1: +3.3V -> Net-(JP11-B)
- J4 pad 1: Net-(J4-Pin_1) -> xbt_B
- J4 pad 2: Net-(J4-Pin_2) -> /+19.5V_raw
- J4 pad 3: Net-(J4-Pin_3) -> /Dout_toComputer
- J4 pad 4: +3.3V -> GND
- J4 pad 5: GND -> xbt_C
- RN1 pad 2: unconnected-(RN1-R1-Pad2) -> relay_reset3
- RN1 pad 3: relay_reset3 -> relay_reset2
- RN1 pad 4: relay_reset2 -> relay_reset1
- RN1 pad 5: relay_reset1 -> relay_cal_res
- RN1 pad 6: relay_cal_res -> relay_cal_cont
- RN1 pad 7: relay_cal_cont -> relay_gnd_cond
- RN1 pad 8: relay_gnd_cond -> relay_xbt8
- RN1 pad 9: relay_xbt8 -> unconnected-(RN1-R8-Pad9)
- RN2 pad 5: SSR_xbt8 -> SSR_xbt7
- RN2 pad 6: SSR_xbt7 -> SSR_xbt6
- RN2 pad 7: SSR_xbt6 -> SSR_xbt8
- RN4 pad 5: SSR_xbt4 -> SSR_xbt3
- RN4 pad 6: SSR_xbt3 -> SSR_xbt2
- RN4 pad 7: SSR_xbt2 -> SSR_xbt4
- U5 pad 6: +3.3V -> Net-(JP11-B)
- U6 pad 10: Net-(J4-Pin_3) -> Enable_M1
- U6 pad 11: Net-(J4-Pin_2) -> Enable_M2
- U6 pad 14: STEP -> Enable_M3
- U6 pad 15: relay_xbt1 -> Enable_M4
- U6 pad 2: Enable_M7 -> SSR_xbt3
- U6 pad 20: relay_xbt2 -> Enable_M5
- U6 pad 21: relay_xbt3 -> Enable_M6
- U6 pad 22: relay_xbt4 -> Enable_M7
- U6 pad 23: relay_xbt5 -> Enable_M8
- U6 pad 24: Net-(J4-Pin_1) -> DIR
- U6 pad 25: Enable_M1 -> /free_pc5
- U6 pad 26: relay_cal_cont -> STEP
- U6 pad 27: relay_cal_res -> Net-(J24-Pin_3)
- U6 pad 28: relay_reset1 -> Net-(J24-Pin_4)
- U6 pad 29: SSR_xbt4 -> /UART3_TX
- U6 pad 3: Enable_M8 -> SSR_xbt2
- U6 pad 30: SSR_xbt5 -> /UART3_RX
- U6 pad 33: SSR_xbt6 -> Net-(J24-Pin_5)
- U6 pad 34: SSR_xbt7 -> Net-(J7-Pin_1)
- U6 pad 35: SSR_xbt8 -> relay_reset3
- U6 pad 36: Net-(J7-Pin_1) -> relay_reset2
- U6 pad 37: Enable_M2 -> relay_reset1
- U6 pad 38: Enable_M3 -> relay_cal_res
- U6 pad 39: Enable_M4 -> relay_cal_cont
- U6 pad 4: DIR -> SSR_xbt1
- U6 pad 40: Enable_M5 -> relay_gnd_cond
- U6 pad 41: relay_xbt6 -> relay_xbt8
- U6 pad 44: relay_xbt7 -> SSR_xbt8
- U6 pad 45: relay_xbt8 -> SSR_xbt7
- U6 pad 50: relay_gnd_cond -> SSR_xbt6
- U6 pad 51: /UART3_TX -> SSR_xbt5
- U6 pad 52: /UART3_RX -> relay_xbt7
- U6 pad 53: Enable_M6 -> relay_xbt6
- U6 pad 54: unconnected-(U6-PD2-Pad54) -> relay_xbt5
- U6 pad 55: relay_reset2 -> relay_xbt4
- U6 pad 56: relay_reset3 -> relay_xbt3
- U6 pad 57: SSR_xbt1 -> relay_xbt2
- U6 pad 61: SSR_xbt2 -> relay_xbt1
- U6 pad 62: SSR_xbt3 -> SSR_xbt4
Routing:
- net Vmotor_out: track 0.00 -> 470.0 mm
- net GND: track 0.00 -> 107.9 mm, vias 0 -> 16
- added copper zone on B.Cu, net GND
Other:
- outline, holes or cut-outs redrawn

Commit message: test pads added, no tracks yet
Parts:
- added A: A, TestPoint:TestPoint_Pad_1.0x1.0mm, F.Cu at (203.0, 100.5)
- added B: B, TestPoint:TestPoint_Pad_1.0x1.0mm, F.Cu at (207.0, 100.5)
- added C: C, TestPoint:TestPoint_Pad_1.0x1.0mm, F.Cu at (211.0, 100.5)
- added DIR: DIR, TestPoint:TestPoint_Pad_1.0x1.0mm, F.Cu at (326.0, 141.0)
- added TP1: Vin-adc, TestPoint:TestPoint_Pad_1.0x1.0mm, F.Cu at (96.0, 119.0)
- added TP13: 12V, TestPoint:TestPoint_Pad_1.0x1.0mm, F.Cu at (90.0, 153.0)
- added TP15: Vref, TestPoint:TestPoint_Pad_1.0x1.0mm, F.Cu at (317.0, 130.0)
- added TP16: 3V3, TestPoint:TestPoint_Pad_1.0x1.0mm, F.Cu at (210.0, 129.0)
- added TP18: GND, TestPoint:TestPoint_Pad_1.0x1.0mm, F.Cu at (326.0, 130.0)
- added TP2: MotorCurrent-adc, TestPoint:TestPoint_Pad_1.0x1.0mm, F.Cu at (77.0, 167.0)
- added TP3: D3V3, TestPoint:TestPoint_Pad_1.0x1.0mm, F.Cu at (151.0, 121.0)
- added TP4: A3V3, TestPoint:TestPoint_Pad_1.0x1.0mm, F.Cu at (145.0, 136.2)
- added TP5: GND, TestPoint:TestPoint_Pad_1.0x1.0mm, F.Cu at (112.0, 146.0)
- added TP6: Vin, TestPoint:TestPoint_Pad_1.0x1.0mm, F.Cu at (87.0, 138.5)
- added TP7: GND, TestPoint:TestPoint_Pad_1.0x1.0mm, F.Cu at (87.0, 133.0)
- added TP8: 3V3, TestPoint:TestPoint_Pad_1.0x1.0mm, F.Cu at (112.0, 134.0)
- added TP9: 5V, TestPoint:TestPoint_Pad_1.0x1.0mm, F.Cu at (85.0, 119.0)
- moved J4 35.6 mm to (59.0, 99.5)
- moved FB1 6.25 mm to (142.0, 141.0)
- moved D1 4.97 mm to (78.1, 138.5)
- moved R4 4.90 mm to (101.1, 119.0)
- moved JP11 2.64 mm to (86.0, 167.3)
- moved C16 2.59 mm to (150.1, 142.0)
- moved RV1 2.55 mm to (322.0, 134.0)
- moved J6 2.42 mm to (144.5, 119.5)
- moved C11 2.16 mm to (159.5, 142.0)
- moved C6 2.12 mm to (149.0, 124.5)
- moved U5 1.97 mm to (81.0, 168.0)
- moved JP4 1.73 mm to (72.7, 168.2)
- moved JP5 1.73 mm to (72.7, 172.2)
- moved C4 1.50 mm to (136.5, 121.5)
- moved C9 1.06 mm to (162.5, 126.5)
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Routing:
- net Vmotor_out: track 470.0 -> 0.00 mm
- net GND: track 107.9 -> 25.5 mm, vias 16 -> 0
- net /+19.5V: track 0.00 -> 39.5 mm
- net Net-(U6-PD1): track 0.00 -> 24.4 mm
- net +3.3V: track 0.00 -> 15.9 mm
- net Net-(U6-PD0): track 0.00 -> 15.4 mm
- net /VDDA: track 0.00 -> 11.0 mm
- net /+19.5V_raw: track 0.00 -> 6.73 mm
Other:
- board text added: "track 0.45 mm 1.3A max 0.6 mm 1.6A"

Commit message: New reorganization on relay drivers and microcontroller pins
Routing:
- net /+19.5V: track 39.5 -> 0.00 mm
- net /+19.5V_raw: track 6.73 -> 0.00 mm
Changed lines of the file:
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@@
     (style (thickness 0.15) (arrow_length 1.27) (text_position_mode 0) (extension_height 0.58642) (extension_offset 0.5) keep_text_aligned)
   )
-  (segment (start 81.489 143.511) (end 81.489 139.115072) (width 1.2) (layer "F.Cu") (net 1))
-  (segment (start 61 156.04) (end 61 154.8462) (width 1.2) (layer "F.Cu") (net 1))
-  (segment (start 81.489 139.115072) (end 80.873928 138.5) (width 1.2) (layer "F.Cu") (net 1))
-  (segment (start 61 154.8462) (end 70.3462 145.5) (width 1.2) (layer "F.Cu") (net 1))
-  (segment (start 80.873928 138.5) (end 80 138.5) (width 1.2) (layer "F.Cu") (net 1))
-  (segment (start 80 138.5) (end 87 138.5) (width 1.2) (layer "F.Cu") (net 1))
-  (segment (start 70.3462 145.5) (end 79.5 145.5) (width 1.2) (layer "F.Cu") (net 1))
-  (segment (start 79.5 145.5) (end 81.489 143.511) (width 1.2) (layer "F.Cu") (net 1))
   (segment (start 148.775 134.999998) (end 142.048335 134.999998) (width 0.15) (layer "F.Cu") (net 2))
   (segment (start 161.074299 129.999998) (end 163.4278 127.646497) (width 0.15) (layer "F.Cu") (net 2))
@@
   (segment (start 144.327798 132.249999) (end 144.327798 132.326665) (width 0.15) (layer "F.Cu") (net 12))
   (segment (start 144.327798 132.249999) (end 144.577798 131.999999) (width 0.15) (layer "F.Cu") (net 12))
-  (segment (start 69.769001 138.0099) (end 70.259101 138.5) (width 1.2) (layer "F.Cu") (net 42))
-  (segment (start 70.259101 138.5) (end 76.2916 138.5) (width 1.2) (layer "F.Cu") (net 42))
   (segment (start 142.8556 138.5) (end 142.8556 140.9793) (width 0.15) (layer "F.Cu") (net 289))
   (segment (start 145.749999 135.5) (end 145 136.249999) (width 0.15) (layer "F.Cu") (net 289))
