File: AOML_AB_3.0/AOML_AB_3.0_reorganized-v1.kicad_sch (KiCad schematic)
At the start: 90 parts, among them J1 Conn_01x04, J2 216550-1, J3 Screw_Terminal_01x04, J4 PH2-08-UA, J5 Screw_Terminal_01x04, J6 Conn_01x03, J7 Screw_Terminal_01x07, SW1 TS02-66-70-BK-160-LCR-D, U1 L7812ABD2T-TR, U2 LM7805MPX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

Commit message: Tracks done manually advanced, led on PB1 added, aux connector removed
Parts:
- removed J4: PH2-08-UA, Connector_PinHeader_2.54mm:PinHeader_2x04_P2.54mm_Vertical, symbol Connector_Generic:Conn_02x04_Counter_Clockwise
- added D7: green, LED_green_0603:LED_B1911PG--20D000514U1930_HVK, symbol Device:LED_Small
- added R47: 220, Resistor_0805:RC0805N_YAG, symbol Device:R_Small
Connections:
- net GND: now also R47.1
- net at U6.27 (PB1): now also D7.2 (A)
- new net: D7.1 (K), R47.2
- no-connect marks 4 -> 3
Other:
- note removed: "Test connector"
- moved on the sheet: J2

Commit message: PCB finished, BOM finished
Parts:
- U4: Digikey (none) -> https://www.digikey.com/en/products/detail/texas-instrument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
Changed lines of the file:
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@@
+      (effects (font (size 1.27 1.27)) hide)
+    )
+    (property "Digikey" "https://www.digikey.com/en/products/detail/texas-instruments/MAX3232EIPWR/968150?s=N4IgTCBcDa4JwDYC0BGOAWAzMlSByAIiALoC%2BQA" (at 52.07 223.52 0)
       (effects (font (size 1.27 1.27)) hide)
     )

Commit message: PCB finished ready to order (no fiducials for assembly), BOM finished
Parts:
- C1: Cost (none) -> 0.1; Part (none) -> CL21B334KBFNNNE
- C10, C14, C3: Cost (none) -> 0.11; Part (none) -> CL21B105KBFNNNE
- C11, C16, C17, C18, C19, C21, C22, C24, C25, C26, C27, C28, C29, C6, C7, C8, C9: Cost (none) -> 0.1; Part (none) -> CL21B104KBCNNNC
- C12, C13: Cost (none) -> 0.39; Part (none) -> ECA-1HM101
- C15: Cost (none) -> 0.1; Part (none) -> CL21B474KBFNNNG
- C2: Cost (none) -> 0.1; Part (none) -> CL21B224KBFNNNE
- C20, C23: Cost (none) -> 0.27; Part (none) -> C0805C200J5GAC7800
- C4: Cost (none) -> 0.1; Part (none) -> 860020572003
- C5: Cost (none) -> 1.23; Part (none) -> EEV-FK1E102Q
- D1: Cost (none) -> 0.37; Part (none) -> B340AE-13
- D2, D3: Cost (none) -> 0.21; Part (none) -> BZT52C3V3-7-F
- D4, D5, D6, D7: value green -> green-led; Cost (none) -> 0.1; Part (none) -> B1911PG--20D000514U1930
- FB1: Cost (none) -> 0.1; Part (none) -> 2508051017Y0
- J1: Cost (none) -> 0.19; Part (none) -> 61300411121
- J2: Cost (none) -> 1.68; Part (none) -> 216550-1
- J3, J5: Cost (none) -> 0.72; Part (none) -> TB001-500-04BE
- J6: Cost (none) -> 0.1; Part (none) -> PH1-03-UA
- J7: Cost (none) -> 0.96; Part (none) -> TB001-500-07BE
- R1: Cost (none) -> 0.1; Part (none) -> RT0805FRE076K8L
- R2: Cost (none) -> 0.1; Part (none) -> RT0805FRE073K3L
- R3: Cost (none) -> 0.1; Part (none) -> RT0805FRE0747KL
- R4: Cost (none) -> 0.1; Part (none) -> RT0805FRE075K1L
- R44: Cost (none) -> 0.1; Digikey (none) -> https://www.digikey.com/en/products/detail/yageo/RC0805FR-1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; Part (none) -> RC0805FR-132KL
- R45: Cost (none) -> 0.1; Digikey (none) -> https://www.digikey.com/en/products/detail/yageo/RC0805JR-0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; Part (none) -> RC0805JR-07560RL
- R46, R47: Cost (none) -> 0.1; Digikey (none) -> https://www.digikey.com/en/products/detail/yageo/RC0805FR-1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; Part (none) -> RC0805FR-13220RL
- R5: Cost (none) -> 0.6; Part (none) -> PE2512FKE070R1L
- R6, R9: Cost (none) -> 0.1; Part (none) -> RT0805FRE0710KL
- R7, R8: Cost (none) -> 0.1; Part (none) -> RT0805FRE074K7L
- SW1: Cost (none) -> 0.14; Part (none) -> PTS526 SK15 SMTR2 LFS
- U1: Cost (none) -> 1.1; Part (none) -> L7812ABD2T-TR
- U2: Cost (none) -> 1.61; Part (none) -> LM7805MPX/NOPB
- U3: Cost (none) -> 0.69; Part (none) -> MCP1825ST-3302E/DB
- U4: Cost (none) -> 1.07; Part (none) -> MAX3232EIPWR
- U5: Cost (none) -> 0.97; Part (none) -> INA213AIDCKR
- U6: Cost (none) -> 7.5; Part (none) -> STM32F103RBT6TR
- U7: Cost (none) -> 0.16; Part (none) -> AT24C01D-STUM-T
- Y1: Cost (none) -> 0.17; Part (none) -> ABLS-8.000MHZ-20-B-3-H-T
